Commit message: Update URDF

File: python/urdf/manip_desc.urdf (robot description, URDF)
Before this commit: robot manip_desc, 6 links, 5 joints
Links:
- removed link p3_link
- removed link r1_link
- added link P3_Link, mass 0.39209; collision mesh filename=meshes/p3_link.stl; visual mesh filename=meshes/p3_link.stl
- added link R1_Link, mass 0.095716; collision mesh filename=meshes/r1_link.stl; visual mesh filename=meshes/r1_link.stl
- added link base_camera_link, mass 0.10321; collision mesh filename=meshes/base_camera_link.stl; visual mesh filename=meshes/base_camera_link.stl
- added link camera_link, mass 0.061767; collision mesh filename=meshes/camera_link.stl; visual mesh filename=meshes/camera_link.stl
- link base_link: mass None -> 0.6413; geometry collision mesh filename=meshes/base_link.stl; visual mesh filename=meshes/base_link.stl
- link r2_link: mass None -> 0.11904; geometry collision mesh filename=meshes/r2_link.stl; visual mesh filename=meshes/r2_link.stl
- link r4_link: mass None -> 0.095715; geometry collision mesh filename=meshes/r4_link.stl; visual mesh filename=meshes/r4_link.stl
- link r5_link: mass None -> 0.095722; geometry collision mesh filename=meshes/r5_link.stl; visual mesh filename=meshes/r5_link.stl
Joints:
- removed joint r1_joint
- removed joint r2_joint
- added joint base_camera_joint: type fixed, parent r5_link, child base_camera_link, origin xyz=-0.0061779 0.023301 -0.072684 rpy=0 0 0, axis 0 0 0
- added joint camera_joint: type fixed, parent base_camera_link, child camera_link, origin xyz=-0.019222 0.04294 -0.028489 rpy=0 0 0, axis 0 0 0
- added joint r1_Joint: type continuous, parent base_link, child r1_link, origin xyz=0 0.2235 0 rpy=0 0 0, axis 0 -1 0
- added joint r2_Joint: type continuous, parent r1_Link, child r2_Link, origin xyz=-0.0058329 0.05 0.047644 rpy=0 0 0, axis 0.12152 0 -0.99259
- joint p3_joint: axis -0.9208 -0.3716 -0.1127 -> -0.92139 -0.3719 -0.1128; limit lower=0.0 upper=0.1 effort=0.1 velocity=0.1 -> lower=-0.1 upper=0.1 effort=0.1 velocity=0.1
- joint r4_joint: axis -0.9208 -0.3716 -0.1127 -> -0.92139 -0.3719 -0.1128; limit lower=-3.1416 upper=3.1416 effort=1 velocity=1 -> (none); type revolute -> continuous
- joint r5_joint: limit lower=-3.1416 upper=3.1416 effort=1 velocity=1 -> (none); type revolute -> continuous
